File: hardware/_autosave-Axis_Basic.kicad_sch (KiCad schematic)
At the start: 58 parts, among them J1 USB_C_Receptacle_USB2.0, J2 JST_PH, J3 JST_PH, J4 S2B-PH-K-S, J5 1175-1628-ND, J6 Conn_01x10, SW1 RKB2SJK, SW2 RKB2SJK, U1 TLV493D, U2 UA78M33CDCYR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

Commit message: PCB layout and routing complete
Connections:
- no-connect marks 14 -> 16
Changed lines of the file:
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@@
   )
   (no_connect (at 40.64 54.61))
+  (no_connect (at 90.17 97.79))
   (no_connect (at 139.7 39.37))
   (no_connect (at 90.17 128.27))
@@
   (no_connect (at 196.85 139.7))
   (no_connect (at 90.17 138.43))
+  (no_connect (at 63.5 109.22))
   (no_connect (at 90.17 102.87))
   (no_connect (at 40.64 57.15))
@@
     (stroke (width 0) (type default))
   )
-  (wire (pts (xy 68.58 97.79) (xy 90.17 97.79))
-    (stroke (width 0) (type default))
-  )
   (wire (pts (xy 186.69 39.37) (xy 182.88 39.37))
     (stroke (width 0) (type default))
@@
     (stroke (width 0) (type default))
   )
-  (wire (pts (xy 68.58 101.6) (xy 68.58 97.79))
-    (stroke (width 0) (type default))
-  )
