File: hardware/Main Board/_autosave-Axis_Basic.kicad_pcb (KiCad board)
At the start: 4 copper layers, 42 x 42 mm, 58 parts, among them J1 USB_C_Receptacle_USB2.0, J2 JST_PH, J3 JST_PH, J4 S2B-PH-K-S, J5 1175-1628-ND, J6 Conn_01x10, SW1 RKB2SJK, SW2 RKB2SJK, U1 TLV493D, U2 UA78M33CDCYR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

Commit message: New rev for base board
Parts:
- J6: value Conn_01x10 -> 1-84952-4; footprint Connector_PinSocket_2.54mm:PinSocket_2x05_P2.54mm_Vertical -> Connector_FFC-FPC:TE_1-84952-4_1x14-1MP_P1.0mm_Horizontal
- moved J6 34.3 mm to (163.9, 100.0)
- moved J1 33.9 mm to (143.5, 83.3), turned to 180 degrees
- moved R13 32.7 mm to (160.0, 110.5), turned to -90 degrees
- moved J3 31.8 mm to (159.5, 84.3), turned to 180 degrees
- moved D7 31.5 mm to (132.8, 90.9)
- moved R11 29.5 mm to (160.0, 108.5), turned to -90 degrees
- moved R12 28.4 mm to (153.8, 110.5), turned to 90 degrees
- moved U5 28.1 mm to (156.7, 110.1), turned to 180 degrees
- moved R1 26.3 mm to (138.6, 88.8), turned to 180 degrees
- moved D1 24.5 mm to (139.6, 92.2), turned to 180 degrees
- moved R6 24.4 mm to (151.1, 118.3)
- moved D4 22.6 mm to (142.4, 89.0), turned to 0 degrees
- moved R9 22.6 mm to (148.2, 106.6), turned to 0 degrees
- moved C3 22.1 mm to (151.1, 117.1), turned to 180 degrees
- moved J5 21.7 mm to (158.7, 113.3), turned to -90 degrees
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Connections:
- J6 pad 10: +3.3V -> ETH_CS
- J6 pad 2: SDA1 -> PA01
- J6 pad 3: ETH_CS -> PA02
- J6 pad 4: SCL1 -> PA03
- J6 pad 5: MISO -> AUX1
- J6 pad 6: unconnected-(J6-Pin_6-Pad6) -> AUX2
- J6 pad 7: SCK -> unconnected-(J6-Pin_7-Pad7)
- J6 pad 8: Net-(J6-Pin_8) -> SDA1
- J6 pad 9: MOSI -> SCL1
- U3 pad 1: unconnected-(U3-PA00/SERCOM1_0-Pad1) -> EN
- U3 pad 15: unconnected-(U3-PA10/SERCOM0_2/SERCOM2_2-Pad15) -> AUX1
- U3 pad 2: Net-(J6-Pin_8) -> PA01
- U3 pad 27: DIR -> NEOPIX
- U3 pad 28: STEP -> AUX2
- U3 pad 3: unconnected-(U3-PA02-Pad3) -> PA02
- U3 pad 30: INDEX -> unconnected-(U3-PA21/SERCOM5_3/SERCOM3_3-Pad30)
- U3 pad 32: MOT_M1 -> unconnected-(U3-PA23/SERCOM3_1/SERCOM5_0-Pad32)
- U3 pad 37: MOT_M0 -> DIR
- U3 pad 38: unconnected-(U3-PB23/SERCOM1_3/SERCOM5_3-Pad38) -> STEP
- U3 pad 39: EN -> INDEX
- U3 pad 4: unconnected-(U3-PA03-Pad4) -> PA03
- U3 pad 47: NEOPIX -> MOT_M1
- U3 pad 48: unconnected-(U3-PB03/SERCOM5_1-Pad48) -> MOT_M0
Routing:
- net GND: track 154.7 -> 84.1 mm, vias 43 -> 31
- net Net-(R5-Pad1): track 48.4 -> 3.20 mm, vias 4 -> 0
- net User_Input: track 80.8 -> 38.7 mm, vias 3 -> 2
- net Net-(J6-Pin_8): track 37.7 -> 0.00 mm, vias 1 -> 0
- net SCL1: track 48.5 -> 14.0 mm
- net DIAG: track 8.38 -> 40.2 mm, vias 0 -> 2
- net SDA1: track 47.6 -> 19.1 mm, vias 2 -> 1
- net ETH_CS: track 32.9 -> 4.49 mm
- net SDA2: track 45.3 -> 17.0 mm, vias 2 -> 0
- net AUX2: track 0.00 -> 28.2 mm, vias 0 -> 2
- net VCC: track 37.0 -> 12.7 mm, vias 13 -> 12
- net EEPROM_CS: track 17.2 -> 37.7 mm
- net SCL2: track 42.0 -> 21.7 mm, vias 2 -> 0
- net AUX1: track 0.00 -> 17.9 mm, vias 0 -> 2
- net SWDIO: track 8.09 -> 22.6 mm
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- removed copper zone on B.Cu, net GND
Other:
- board text added: "-"
- board text added: "12v"
- board text added: "GND"
- board text added: "RST"
- board text added: "SCL"
- board text added: "SDA"
