File: hardware/Main Board/_autosave-Axis_Basic.kicad_pcb (KiCad board)
At the start: 4 copper layers, 42 x 42 mm, 78 parts, among them J1 USB4105-GF-A, J2 JST_PH, J3 JST_SH, J4 S2B-PH-K-S, J5 JST_SH, J6 1-84952-4, SW1 RKB2SJK, SW2 RKB2SJK, U1 TLV493D, U2 UA78M33CDCYR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

Commit message: PCB V1.0.0 Ordered
Routing:
- net GND: vias 102 -> 100
Other:
- board text added: "I2C"
Changed lines of the file:
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@@
+		)
+	)
+	(gr_text "I2C"
+		(at 162.6 120.5 0)
+		(layer "F.SilkS")
+		(effects
+			(font
+				(size 1.5 1.5)
+				(thickness 0.3)
+				(bold yes)
+			)
+			(justify left bottom)
 		)
 	)
@@
 	)
 	(via
-		(at 164 120)
-		(size 0.7)
-		(drill 0.35)
-		(layers "F.Cu" "B.Cu")
-		(free yes)
-		(net 2)
-	)
-	(via
 		(at 137.1 92.3)
 		(size 0.7)
@@
 		(size 0.7)
 		(drill 0.35)
-		(layers "F.Cu" "B.Cu")
-		(free yes)
-		(net 2)
-	)
-	(via
-		(at 166 120)
-		(size 0.7)
-		(drill 0.35)
